File: hardware/sd_karte.sch (KiCad schematic (older format))
At the start: 11 parts

Commit message: Hardware Projekt knovertiert von KiCad 4 -> KiCad 5 - Schaltplan angepasst - neues Detailfoto hinzugefügt - Footprints neu zugeordnet, somit ist auch wieder eine 3D Darstellung möglich - Readme.md angepasst
Parts:
- removed SD1: ATTEND_104H-TDA0-R01, ka_sd_sockets:ATTEND_104H-TDA0-R01, symbol ATTEND_104H-TDA0-R01
- added SD1: ATTEND_104H-TDA0-R01, sd_sockets_tk:ATTEND_104H-TDA0-R01, symbol sd_sockets_tk:ATTEND_104H-TDA0-R01
- D1, D2: footprint Diodes_THT:D_DO-35_SOD27_P7.62mm_Horizontal -> Diode_THT:D_DO-35_SOD27_P7.62mm_Horizontal; symbol D -> Diode:1N4148
- R2, R4, R5, R6, R7, R8, R9: footprint Discret:R4-5 -> Resistor_THT:R_Axial_DIN0207_L6.3mm_D2.5mm_P10.16mm_Horizontal; symbol R -> Device:R
- R3: value 47kR -> 47k; footprint Discret:R4-5 -> Resistor_THT:R_Axial_DIN0207_L6.3mm_D2.5mm_P10.16mm_Horizontal; symbol R -> Device:R
Connections:
- net GND: now also SD1.3 (VSS1), SD1.6 (VSS2), SD1.G (GND), SD1.Sc (Common_Pin)
- net MISO: now also SD1.7 (DAT0)
- net SD_DETECT: now also SD1.Cd (Card_Detection)
- net SD_WP: now also SD1.Wp (Write_Protection)
- net at D1.1 (K): now also SD1.4 (VDD)
- net at R4.2, R7.1: now also SD1.1 (DAT3/CS/CD)
- net at R5.2, R8.1: now also SD1.2 (CMD)
- net at R6.2, R9.1: now also SD1.5 (CLK)
Other:
- moved on the sheet: R2, R3
Changed lines of the file:
@@
-EESchema Schematic File Version 2
-LIBS:power
-LIBS:1541-rebuild-rescue
-LIBS:device
-LIBS:transistors
-LIBS:conn
-LIBS:linear
-LIBS:regul
-LIBS:74xx
-LIBS:cmos4000
-LIBS:adc-dac
-LIBS:memory
-LIBS:xilinx
-LIBS:microcontrollers
-LIBS:dsp
-LIBS:microchip
-LIBS:analog_switches
-LIBS:motorola
-LIBS:texas
-LIBS:intel
-LIBS:audio
-LIBS:interface
-LIBS:digital-audio
-LIBS:philips
-LIBS:display
-LIBS:cypress
-LIBS:siliconi
-LIBS:opto
-LIBS:atmel
-LIBS:contrib
-LIBS:valves
-LIBS:Oscillators
-LIBS:w_analog
-LIBS:w_connectors
-LIBS:w_device
-LIBS:w_logic
-LIBS:w_memory
-LIBS:w_microcontrollers
-LIBS:w_opto
-LIBS:w_relay
-LIBS:w_rtx
-LIBS:w_transistor
-LIBS:w_vacuum
-LIBS:ka_sd_sockets
+EESchema Schematic File Version 4
 LIBS:1541-rebuild-cache
-EELAYER 25 0
+EELAYER 30 0
 EELAYER END
 $Descr A4 11693 8268
@@
 Sheet 2 4
 Title "1541-rebuid"
-Date "2018-05-16"
-Rev "1.3.5"
+Date "2020-04-14"
+Rev "1.4.0"
 Comp ""
 Comment1 "Erstellt von: Thorsten Kattanek"
@@
 $EndDescr
 $Comp
-L D D1
+L Diode:1N4148 D1
 U 1 1 55F7A3CC
 P 4450 4050
 F 0 "D1" H 4450 4150 50  0000 C CNN
 F 1 "1N4148" H 4450 3950 50  0000 C CNN
-F 2 "Diodes_THT:D_DO-35_SOD27_P7.62mm_Horizontal" H 4450 4050 60  0001 C CNN
+F 2 "Diode_THT:D_DO-35_SOD27_P7.62mm_Horizontal" H 4450 4050 60  0001 C CNN
 F 3 "" H 4450 4050 60  0000 C CNN
 	1    4450 4050
@@
 $EndComp
 $Comp
-L D D2
+L Diode:1N4148 D2
 U 1 1 55F7A4EB
 P 4450 4450
 F 0 "D2" H 4450 4550 50  0000 C CNN
 F 1 "1N4148" H 4450 4350 50  0000 C CNN
-F 2 "Diodes_THT:D_DO-35_SOD27_P7.62mm_Horizontal" H 4450 4450 60  0001 C CNN
+F 2 "Diode_THT:D_DO-35_SOD27_P7.62mm_Horizontal" H 4450 4450 60  0001 C CNN
 F 3 "" H 4450 4450 60  0000 C CNN
 	1    4450 4450
@@
 $EndComp
 $Comp
-L +5V #PWR015
+L power:+5V #PWR015
 U 1 1 55F7A887
 P 4450 4700
@@
 NoConn ~ 4800 3050
 $Comp
-L R R7
+L Device:R R7
 U 1 1 55F7B36C
 P 3700 3150
 F 0 "R7" V 3600 3150 50  0000 C CNN
 F 1 "1,8k" V 3700 3150 50  0000 C CNN
-F 2 "Discret:R4-5" V 3630 3150 30  0001 C CNN
+F 2 "Resistor_THT:R_Axial_DIN0207_L6.3mm_D2.5mm_P10.16mm_Horizontal" V 3630 3150 30  0001 C CNN
 F 3 "" H 3700 3150 30  0000 C CNN
 	1    3700 3150
@@
 $EndComp
 $Comp
-L R R8
+L Device:R R8
 U 1 1 55F7B401
 P 3900 3250
 F 0 "R8" V 3980 3250 50  0000 C CNN
 F 1 "1,8k" V 3900 3250 50  0000 C CNN
-F 2 "Discret:R4-5" V 3830 3250 30  0001 C CNN
+F 2 "Resistor_THT:R_Axial_DIN0207_L6.3mm_D2.5mm_P10.16mm_Horizontal" V 3830 3250 30  0001 C CNN
 F 3 "" H 3900 3250 30  0000 C CNN
 	1    3900 3250
@@
 $EndComp
 $Comp
-L R R9
+L Device:R R9
 U 1 1 55F7B48C
 P 3700 3550
 F 0 "R9" V 3780 3550 50  0000 C CNN
 F 1 "1,8k" V 3700 3550 50  0000 C CNN
-F 2 "Discret:R4-5" V 3630 3550 30  0001 C CNN
+F 2 "Resistor_THT:R_Axial_DIN0207_L6.3mm_D2.5mm_P10.16mm_Horizontal" V 3630 3550 30  0001 C CNN
 F 3 "" H 3700 3550 30  0000 C CNN
 	1    3700 3550
@@
 $EndComp
 $Comp
-L R R4
+L Device:R R4
 U 1 1 55F7BA6C
 P 3900 2900
 F 0 "R4" V 3980 2900 50  0000 C CNN
 F 1 "3,3k" V 3900 2900 50  0000 C CNN
-F 2 "Discret:R4-5" V 3830 2900 30  0001 C CNN
+F 2 "Resistor_THT:R_Axial_DIN0207_L6.3mm_D2.5mm_P10.16mm_Horizontal" V 3830 2900 30  0001 C CNN
 F 3 "" H 3900 2900 30  0000 C CNN
 	1    3900 2900
@@
 $EndComp
 $Comp
-L R R5
+L Device:R R5
 U 1 1 55F7BC20
 P 4100 2900
 F 0 "R5" V 4180 2900 50  0000 C CNN
 F 1 "3,3k" V 4100 2900 50  0000 C CNN
-F 2 "Discret:R4-5" V 4030 2900 30  0001 C CNN
+F 2 "Resistor_THT:R_Axial_DIN0207_L6.3mm_D2.5mm_P10.16mm_Horizontal" V 4030 2900 30  0001 C CNN
 F 3 "" H 4100 2900 30  0000 C CNN
 	1    4100 2900
@@
 $EndComp
 $Comp
-L R R6
+L Device:R R6
 U 1 1 55F7BCCD
 P 4300 2900
 F 0 "R6" V 4380 2900 50  0000 C CNN
 F 1 "3,3k" V 4300 2900 50  0000 C CNN
-F 2 "Discret:R4-5" V 4230 2900 30  0001 C CNN
+F 2 "Resistor_THT:R_Axial_DIN0207_L6.3mm_D2.5mm_P10.16mm_Horizontal" V 4230 2900 30  0001 C CNN
 F 3 "" H 4300 2900 30  0000 C CNN
 	1    4300 2900
@@
 	3250 3150 3550 3150
 Wire Wire Line
-	3850 3150 4800 3150
-Wire Wire Line
-	4050 3250 4800 3250
+	3850 3150 3900 3150
+Wire Wire Line
+	4050 3250 4100 3250
 Wire Wire Line
 	3750 3250 3250 3250
@@
 	3250 3550 3550 3550
 Wire Wire Line
-	3850 3550 4800 3550
+	3850 3550 4300 3550
 Wire Wire Line
 	3900 3050 3900 3150
@@
 Connection ~ 4300 3550
 Wire Wire Line
-	4100 2500 4100 2750
+	4100 2500 4100 2600
 Wire Wire Line
 	4300 2600 4300 2750
 Wire Wire Line
-	3900 2600 4300 2600
+	3900 2600 4100 2600
 Connection ~ 4100 2600
 Wire Wire Line
@@
 	4800 3350 4700 3350
 Wire Wire Line
-	4700 3350 4700 3900
+	4700 3350 4700 3650
 Wire Wire Line
 	4800 3650 4700 3650
 Connection ~ 4700 3650
 $Comp
-L R R2
+L Device:R R2
 U 1 1 5ADB73A5
-P 6650 2750
-F 0 "R2" V 6730 2750 50  0000 C CNN
-F 1 "47k" V 6650 2750 50  0000 C CNN
-F 2 "Discret:R4-5" V 6580 2750 50  0001 C CNN
-F 3 "" H 6650 2750 50  0001 C CNN
-	1    6650 2750
-	1    0    0    -1
-$EndComp
-$Comp
-L R R3
+P 6650 2700
+F 0 "R2" V 6730 2700 50  0000 C CNN
+F 1 "47k" V 6650 2700 50  0000 C CNN
+F 2 "Resistor_THT:R_Axial_DIN0207_L6.3mm_D2.5mm_P10.16mm_Horizontal" V 6580 2700 50  0001 C CNN
+F 3 "" H 6650 2700 50  0001 C CNN
+	1    6650 2700
+	1    0    0    -1
+$EndComp
+$Comp
+L Device:R R3
 U 1 1 5ADB753C
-P 6900 2750
-F 0 "R3" V 6980 2750 50  0000 C CNN
-F 1 "47kR" V 6900 2750 50  0000 C CNN
-F 2 "Discret:R4-5" V 6830 2750 50  0001 C CNN
-F 3 "" H 6900 2750 50  0001 C CNN
-	1    6900 2750
-	1    0    0    -1
-$EndComp
-$Comp
-L +5V #PWR016
+P 6900 2700
+F 0 "R3" V 6980 2700 50  0000 C CNN
+F 1 "47k" V 6900 2700 50  0000 C CNN
+F 2 "Resistor_THT:R_Axial_DIN0207_L6.3mm_D2.5mm_P10.16mm_Horizontal" V 6830 2700 50  0001 C CNN
+F 3 "" H 6900 2700 50  0001 C CNN
+	1    6900 2700
+	1    0    0    -1
+$EndComp
+$Comp
+L power:+5V #PWR016
 U 1 1 5ADB75CA
-P 6650 2400
-F 0 "#PWR016" H 6650 2250 50  0001 C CNN
-F 1 "+5V" H 6650 2540 50  0000 C CNN
-F 2 "" H 6650 2400 60  0000 C CNN
-F 3 "" H 6650 2400 60  0000 C CNN
-	1    6650 2400
-	1    0    0    -1
-$EndComp
-Wire Wire Line
-	6650 2400 6650 2600
-Wire Wire Line
-	6650 2500 6900 2500
-Wire Wire Line
-	6900 2500 6900 2600
-Connection ~ 6650 2500
+P 6650 2350
+F 0 "#PWR016" H 6650 2200 50  0001 C CNN
+F 1 "+5V" H 6650 2490 50  0000 C CNN
+F 2 "" H 6650 2350 60  0000 C CNN
+F 3 "" H 6650 2350 60  0000 C CNN
+	1    6650 2350
+	1    0    0    -1
+$EndComp
+Wire Wire Line
+	6650 2350 6650 2450
+Wire Wire Line
+	6650 2450 6900 2450
+Wire Wire Line
+	6900 2450 6900 2550
+Connection ~ 6650 2450
 Text HLabel 7150 3150 2    60   Input ~ 0
 SD_DETECT
@@
 SD_WP
 Wire Wire Line
-	6500 3050 7150 3050
-Wire Wire Line
-	7150 3150 6500 3150
-Wire Wire Line
-	6650 2900 6650 3050
+	6500 3050 6650 3050
+Wire Wire Line
+	7150 3150 6900 3150
+Wire Wire Line
+	6650 2850 6650 3050
 Connection ~ 6650 3050
 Wire Wire Line
-	6900 2900 6900 3150
+	6900 2850 6900 3150
 Connection ~ 6900 3150
 Text Notes 650  7650 0    60   ~ 0
 SD_DETECT ist LO wenn eine Karte eingestekt ist\nSD_WP ist LO wenn Schreibschutz aktiv\n(SD_WP muss HI sein damit man schreiben kann)
 $Comp
-L GND #PWR017
+L power:GND #PWR017
 U 1 1 5AF0D189
 P 4100 2500
@@
 $EndComp
 $Comp
-L GND #PWR018
+L power:GND #PWR018
 U 1 1 5AF0D222
 P 4700 3900
@@
 $EndComp
 Wire Wire Line
-	6500 3250 6550 3250
-Wire Wire Line
-	6550 3250 6550 3900
-Wire Wire Line
-	6550 3850 6500 3850
-$Comp
-L GND #PWR019
+	6500 3250 6700 3250
+Wire Wire Line
+	6700 3250 6700 3850
+Wire Wire Line
+	6700 3850 6500 3850
+$Comp
+L power:GND #PWR019
 U 1 1 5AF0AE1C
-P 6550 3900
-F 0 "#PWR019" H 6550 3650 50  0001 C CNN
-F 1 "GND" H 6550 3750 50  0000 C CNN
-F 2 "" H 6550 3900 50  0001 C CNN
-F 3 "" H 6550 3900 50  0001 C CNN
-	1    6550 3900
-	1    0    0    -1
-$EndComp
-Connection ~ 6550 3850
-$Comp
-L ATTEND_104H-TDA0-R01 SD1
-U 1 1 5AF5BDB3
+P 6700 4000
+F 0 "#PWR019" H 6700 3750 50  0001 C CNN
+F 1 "GND" H 6700 3850 50  0000 C CNN
+F 2 "" H 6700 4000 50  0001 C CNN
+F 3 "" H 6700 4000 50  0001 C CNN
+	1    6700 4000
+	1    0    0    -1
+$EndComp
+Connection ~ 6700 3850
+Wire Wire Line
+	3900 3150 4800 3150
+Wire Wire Line
+	4100 3250 4800 3250
+Wire Wire Line
+	4300 3550 4800 3550
+Wire Wire Line
+	4100 2600 4100 2750
+Wire Wire Line
+	4100 2600 4300 2600
+Wire Wire Line
+	4700 3650 4700 3900
+Wire Wire Line
+	6650 2450 6650 2550
+Wire Wire Line
+	6650 3050 7150 3050
+Wire Wire Line
+	6900 3150 6500 3150
+Wire Wire Line
+	6700 3850 6700 4000
+$Comp
+L sd_sockets_tk:ATTEND_104H-TDA0-R01 SD1
+U 1 1 5E94FB8A
 P 5650 3450
-F 0 "SD1" H 5650 3950 60  0000 C CNN
-F 1 "ATTEND_104H-TDA0-R01" H 5650 2950 60  0000 C CNN
-F 2 "ka_sd_sockets:ATTEND_104H-TDA0-R01" H 3800 2100 60  0001 C CNN
+F 0 "SD1" H 5650 4097 60  0000 C CNN
+F 1 "ATTEND_104H-TDA0-R01" H 5650 3991 60  0000 C CNN
+F 2 "sd_sockets_tk:ATTEND_104H-TDA0-R01" H 3800 2100 60  0001 C CNN
 F 3 "" H 3800 2100 60  0001 C CNN
 	1    5650 3450
